Commit message: feat(rover_description): real-mass correction, materials, motor velocity limit
Chassis 9.78->41.71 kg (internals absent from CAD; inertia scaled), total 59.06 kg. Palette matched to real rover. Wheel velocity 28 rad/s from AK10-9 KV100. Steer +/-90 confirmed, R_min 0.417 m FINAL. Launch embeds GZ_SIM_RESOURCE_PATH.

Refs: T0-R1, SURA-21

File: src/rover_description/urdf/karasimsekURDF.urdf.xacro (robot description, xacro)
@@ -11,5 +11,5 @@
   <xacro:property name="steer_velocity"      value="2.0"/>
   <!-- Wheel spin limits (about +Y) -->
-  <xacro:property name="wheel_velocity"      value="50.0"/>
+  <xacro:property name="wheel_velocity"      value="28.0"/>
   <xacro:arg name="diff_joints" default="fixed"/>
   <xacro:property name="diff_activation"    value="$(arg diff_joints)"/> <!--set 'revolute' to enable differential bar motion -->
@@ -45,7 +45,7 @@
     <inertial>
       <origin xyz="0.011561 -0.031261 0.11152" rpy="0 0 0"/>
-      <mass value="9.7774"/>
-      <inertia ixx="0.41887" ixy="-0.00010081" ixz="1.9651E-06"
-               iyy="0.22572" iyz="-0.0056869"  izz="0.58468"/>
+      <mass value="41.71"/>
+      <inertia ixx="1.786883" ixy="-0.000430" ixz="0.000008"
+               iyy="0.962913" iyz="-0.024260"  izz="2.494222"/>
     </inertial>
     <visual>
@@ -54,7 +54,5 @@
         <mesh filename="package://rover_description/meshes/Chassis_link.STL"/>
       </geometry>
-      <material name="">
-        <color rgba="0.79216 0.81961 0.93333 1"/>
-      </material>
+      <material name="carbon_dark"><color rgba="0.13 0.13 0.15 1"/></material>
     </visual>
     <collision>
@@ -84,7 +82,5 @@
         <mesh filename="package://rover_description/meshes/left_link.STL"/>
       </geometry>
-      <material name="">
-        <color rgba="0.792156862745098 0.819607843137255 0.933333333333333 1"/>
-      </material>
+      <material name="gunmetal"><color rgba="0.28 0.29 0.32 1"/></material>
     </visual>
     <collision>
@@ -115,7 +111,5 @@
         <mesh filename="package://rover_description/meshes/FLSteer_Link.STL"/>
       </geometry>
-      <material name="">
-        <color rgba="0.792156862745098 0.819607843137255 0.933333333333333 1"/>
-      </material>
+      <material name="alu_bright"><color rgba="0.78 0.79 0.81 1"/></material>
     </visual>
   </link>
@@ -141,7 +135,5 @@
         <mesh filename="package://rover_description/meshes/FLWheel_Link.STL"/>
       </geometry>
-      <material name="">
-        <color rgba="0.792156862745098 0.819607843137255 0.933333333333333 1"/>
-      </material>
+      <material name="tire_black"><color rgba="0.05 0.05 0.05 1"/></material>
     </visual>
     <collision>
@@ -173,7 +165,5 @@
         <mesh filename="package://rover_description/meshes/RLSteer_Link.STL"/>
       </geometry>
-      <material name="">
-        <color rgba="0.792156862745098 0.819607843137255 0.933333333333333 1"/>
-      </material>
+      <material name="alu_bright"><color rgba="0.78 0.79 0.81 1"/></material>
     </visual>
   </link>
@@ -199,7 +189,5 @@
         <mesh filename="package://rover_description/meshes/RLWheel_Link.STL"/>
       </geometry>
-      <material name="">
-        <color rgba="0.792156862745098 0.819607843137255 0.933333333333333 1"/>
-      </material>
+      <material name="tire_black"><color rgba="0.05 0.05 0.05 1"/></material>
     </visual>
     <collision>
@@ -231,7 +219,5 @@
         <mesh filename="package://rover_description/meshes/LeftRod_Link.STL"/>
       </geometry>
-      <material name="">
-        <color rgba="0.792156862745098 0.819607843137255 0.933333333333333 1"/>
-      </material>
+      <material name="alu_silver"><color rgba="0.75 0.76 0.78 1"/></material>
     </visual>
   </link>
@@ -253,7 +239,5 @@
         <mesh filename="package://rover_description/meshes/FirstBall_Link.STL"/>
       </geometry>
-      <material name="">
-        <color rgba="0.529411764705882 0.549019607843137 0.549019607843137 1"/>
-      </material>
+      <material name="joint_black"><color rgba="0.10 0.10 0.10 1"/></material>
     </visual>
   </link>
@@ -275,7 +259,5 @@
         <mesh filename="package://rover_description/meshes/SecondBall_Link.STL"/>
       </geometry>
-      <material name="">
-        <color rgba="0.529411764705882 0.549019607843137 0.549019607843137 1"/>
-      </material>
+      <material name="joint_black"><color rgba="0.10 0.10 0.10 1"/></material>
     </visual>
   </link>
@@ -297,7 +279,5 @@
         <mesh filename="package://rover_description/meshes/right_link.STL"/>
       </geometry>
-      <material name="">
-        <color rgba="0.792156862745098 0.819607843137255 0.933333333333333 1"/>
-      </material>
+      <material name="gunmetal"><color rgba="0.28 0.29 0.32 1"/></material>
     </visual>
     <collision>
@@ -328,7 +308,5 @@
         <mesh filename="package://rover_description/meshes/FRSteer_Link.STL"/>
       </geometry>
-      <material name="">
-        <color rgba="0.792156862745098 0.819607843137255 0.933333333333333 1"/>
-      </material>
+      <material name="alu_bright"><color rgba="0.78 0.79 0.81 1"/></material>
     </visual>
   </link>
@@ -354,7 +332,5 @@
         <mesh filename="package://rover_description/meshes/FRWheel_Link.STL"/>
       </geometry>
-      <material name="">
-        <color rgba="0.792156862745098 0.819607843137255 0.933333333333333 1"/>
-      </material>
+      <material name="tire_black"><color rgba="0.05 0.05 0.05 1"/></material>
     </visual>
     <collision>
@@ -386,7 +362,5 @@
         <mesh filename="package://rover_description/meshes/RRSteer_Link.STL"/>
       </geometry>
-      <material name="">
-        <color rgba="0.792156862745098 0.819607843137255 0.933333333333333 1"/>
-      </material>
+      <material name="alu_bright"><color rgba="0.78 0.79 0.81 1"/></material>
     </visual>
   </link>
@@ -412,7 +386,5 @@
         <mesh filename="package://rover_description/meshes/RRWheel_Link.STL"/>
       </geometry>
-      <material name="">
-        <color rgba="0.792156862745098 0.819607843137255 0.933333333333333 1"/>
-      </material>
+      <material name="tire_black"><color rgba="0.05 0.05 0.05 1"/></material>
     </visual>
     <collision>
@@ -444,7 +416,5 @@
         <mesh filename="package://rover_description/meshes/RightRod_Link.STL"/>
       </geometry>
-      <material name="">
-        <color rgba="0.792156862745098 0.819607843137255 0.933333333333333 1"/>
-      </material>
+      <material name="alu_silver"><color rgba="0.75 0.76 0.78 1"/></material>
     </visual>
   </link>
@@ -466,7 +436,5 @@
         <mesh filename="package://rover_description/meshes/RearRightBall_Link.STL"/>
       </geometry>
-      <material name="">
-        <color rgba="0.529411764705882 0.549019607843137 0.549019607843137 1"/>
-      </material>
+      <material name="joint_black"><color rgba="0.10 0.10 0.10 1"/></material>
     </visual>
   </link>
@@ -488,7 +456,5 @@
         <mesh filename="package://rover_description/meshes/RearRightSecondBall_Link.STL"/>
       </geometry>
-      <material name="">
-        <color rgba="0.529411764705882 0.549019607843137 0.549019607843137 1"/>
-      </material>
+      <material name="joint_black"><color rgba="0.10 0.10 0.10 1"/></material>
     </visual>
   </link>
@@ -510,7 +476,5 @@
         <mesh filename="package://rover_description/meshes/Zed_Link.STL"/>
       </geometry>
-      <material name="">
-        <color rgba="0.627450980392157 0.627450980392157 0.627450980392157 1"/>
-      </material>
+      <material name="zed_navy"><color rgba="0.10 0.12 0.20 1"/></material>
     </visual>
   </link>

Commit message: fix(description): machined-aluminum tone for steer/linkage materials (visual only, rgba); 3/4 front verification frame
No geometry, joints, inertials, or collisions touched. Xacro validated,
joint tree and total mass verified unchanged.

File: src/rover_description/urdf/karasimsekURDF.urdf.xacro (robot description, xacro)
@@ -111,5 +111,5 @@
         <mesh filename="package://rover_description/meshes/FLSteer_Link.STL"/>
       </geometry>
-      <material name="alu_bright"><color rgba="0.78 0.79 0.81 1"/></material>
+      <material name="alu_bright"><color rgba="0.45 0.46 0.48 1"/></material>
     </visual>
   </link>
@@ -165,5 +165,5 @@
         <mesh filename="package://rover_description/meshes/RLSteer_Link.STL"/>
       </geometry>
-      <material name="alu_bright"><color rgba="0.78 0.79 0.81 1"/></material>
+      <material name="alu_bright"><color rgba="0.45 0.46 0.48 1"/></material>
     </visual>
   </link>
@@ -219,5 +219,5 @@
         <mesh filename="package://rover_description/meshes/LeftRod_Link.STL"/>
       </geometry>
-      <material name="alu_silver"><color rgba="0.75 0.76 0.78 1"/></material>
+      <material name="alu_silver"><color rgba="0.42 0.43 0.45 1"/></material>
     </visual>
   </link>
@@ -308,5 +308,5 @@
         <mesh filename="package://rover_description/meshes/FRSteer_Link.STL"/>
       </geometry>
-      <material name="alu_bright"><color rgba="0.78 0.79 0.81 1"/></material>
+      <material name="alu_bright"><color rgba="0.45 0.46 0.48 1"/></material>
     </visual>
   </link>
@@ -362,5 +362,5 @@
         <mesh filename="package://rover_description/meshes/RRSteer_Link.STL"/>
       </geometry>
-      <material name="alu_bright"><color rgba="0.78 0.79 0.81 1"/></material>
+      <material name="alu_bright"><color rgba="0.45 0.46 0.48 1"/></material>
     </visual>
   </link>
@@ -416,5 +416,5 @@
         <mesh filename="package://rover_description/meshes/RightRod_Link.STL"/>
       </geometry>
-      <material name="alu_silver"><color rgba="0.75 0.76 0.78 1"/></material>
+      <material name="alu_silver"><color rgba="0.42 0.43 0.45 1"/></material>
     </visual>
   </link>
